File: IIGS-audio.kicad_sch (KiCad schematic)
At the start: 39 parts, among them J1 Conn_01x07, J2 Conn_01x02_Male, J3 SJ1-3515N, J4 AppleII_slot

Commit message: Upgraded KiCad
Parts:
- U1: value (none) -> 74HC4052D
- U2: value (none) -> TL074
Changed lines of the file:
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@@
     (in_bom yes) (on_board yes) (fields_autoplaced)
     (property "Reference" "U2" (id 0) (at 189.23 87.63 0))
-    (property "Value" "" (id 1) (at 189.23 90.17 0))
+    (property "Value" "TL074" (id 1) (at 189.23 90.17 0))
     (property "Footprint" "Package_SO:SOIC-14_3.9x8.7mm_P1.27mm" (id 2) (at 187.96 95.25 0)
       (effects (font (size 1.27 1.27)) hide)
@@
     (in_bom yes) (on_board yes) (fields_autoplaced)
     (property "Reference" "U2" (id 0) (at 189.23 46.99 0))
-    (property "Value" "" (id 1) (at 189.23 49.53 0))
+    (property "Value" "TL074" (id 1) (at 189.23 49.53 0))
     (property "Footprint" "Package_SO:SOIC-14_3.9x8.7mm_P1.27mm" (id 2) (at 187.96 54.61 0)
       (effects (font (size 1.27 1.27)) hide)
@@
     (in_bom yes) (on_board yes) (fields_autoplaced)
     (property "Reference" "U2" (id 0) (at 151.13 85.09 0))
-    (property "Value" "" (id 1) (at 151.13 87.63 0))
+    (property "Value" "TL074" (id 1) (at 151.13 87.63 0))
     (property "Footprint" "Package_SO:SOIC-14_3.9x8.7mm_P1.27mm" (id 2) (at 149.86 92.71 0)
       (effects (font (size 1.27 1.27)) hide)
@@
     (in_bom yes) (on_board yes)
     (property "Reference" "U1" (id 0) (at 87.63 72.39 0))
-    (property "Value" "" (id 1) (at 87.63 60.96 0))
+    (property "Value" "74HC4052D" (id 1) (at 87.63 60.96 0))
     (property "Footprint" "SOIC127P600X175-16N" (id 2) (at 96.52 62.23 0)
       (effects (font (size 1.27 1.27)) (justify left) hide)
@@
     (in_bom yes) (on_board yes) (fields_autoplaced)
     (property "Reference" "U2" (id 0) (at 151.13 44.45 0))
-    (property "Value" "" (id 1) (at 151.13 46.99 0))
+    (property "Value" "TL074" (id 1) (at 151.13 46.99 0))
     (property "Footprint" "Package_SO:SOIC-14_3.9x8.7mm_P1.27mm" (id 2) (at 149.86 52.07 0)
       (effects (font (size 1.27 1.27)) hide)
@@
       (effects (font (size 1.27 1.27)) (justify left))
     )
-    (property "Value" "" (id 1) (at 250.19 135.8899 0)
+    (property "Value" "TL074" (id 1) (at 250.19 135.8899 0)
       (effects (font (size 1.27 1.27)) (justify left))
     )
