File: IIGS-audio.kicad_pcb (KiCad board)
At the start: 2 copper layers, 65.8 x 46.6 mm, 39 parts, among them J1 Conn_01x07, J2 Conn_01x02_Male, J3 SJ1-3515N, J4 AppleII_slot, U1 74HC4052D, U2 TL074

Commit message: Changed silkscreen label from J-25 to J25 to match the IIGS motherboard
Other:
- board text added: "<-Out to J25"
- board text removed: "<-Out to J-25"
Changed lines of the file:
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@@
     (effects (font (size 1 1) (thickness 0.15)))
   )
-  (gr_text "<-Out to J-25" (at 122.682 119.7585) (layer "F.SilkS")
+  (gr_text "<-Out to J25" (at 122.682 119.7585) (layer "F.SilkS")
     (effects (font (size 1.5 1.5) (thickness 0.3)))
   )
